File: src/lsm6dso-breakout.brd (EAGLE design)
At the start: 18 x 10.6 mm, 5 parts, among them J1 PTH VERT MALE, J2 PTH VERT MALE, U1 LSM6DSOTR

Commit message: Update CAM files.
Parts:
- U1: device _sensors:QFN50P300X250X86-14N -> _sensors:QFN50P250X300X86-14N
Routing:
- net INT1: track 12.3 -> 13.1 mm
Other:
- board text added: "Rev 2"
- board text removed: "Rev 1"
